Commit message: Update test cases

File: models/kuka_lbr.urdf (robot description, URDF)
Before this commit: robot kuka_lbr, 59 links, 58 joints
Joints:
- joint kuka_lbr_l_finger_1_joint_0: type revolute -> fixed
- joint kuka_lbr_l_finger_1_joint_1: type revolute -> fixed
- joint kuka_lbr_l_finger_1_joint_2: type revolute -> fixed
- joint kuka_lbr_l_finger_1_joint_3: type revolute -> fixed
- joint kuka_lbr_l_finger_2_joint_0: type revolute -> fixed
- joint kuka_lbr_l_finger_2_joint_1: type revolute -> fixed
- joint kuka_lbr_l_finger_2_joint_2: type revolute -> fixed
- joint kuka_lbr_l_finger_2_joint_3: type revolute -> fixed
- joint kuka_lbr_l_finger_middle_joint_1: type revolute -> fixed
- joint kuka_lbr_l_finger_middle_joint_2: type revolute -> fixed
- joint kuka_lbr_l_finger_middle_joint_3: type revolute -> fixed
- joint kuka_lbr_r_finger_1_joint_0: type revolute -> fixed
- joint kuka_lbr_r_finger_1_joint_1: type revolute -> fixed
- joint kuka_lbr_r_finger_1_joint_2: type revolute -> fixed
- joint kuka_lbr_r_finger_1_joint_3: type revolute -> fixed
- joint kuka_lbr_r_finger_2_joint_0: type revolute -> fixed
- joint kuka_lbr_r_finger_2_joint_1: type revolute -> fixed
- joint kuka_lbr_r_finger_2_joint_2: type revolute -> fixed
- joint kuka_lbr_r_finger_2_joint_3: type revolute -> fixed
- joint kuka_lbr_r_finger_middle_joint_1: type revolute -> fixed
- joint kuka_lbr_r_finger_middle_joint_2: type revolute -> fixed
- joint kuka_lbr_r_finger_middle_joint_3: type revolute -> fixed
