Commit message: Update examples

File: models/rh5v2/urdf/rh5v2_hybrid.urdf (robot description, URDF)
Before this commit: robot RH5v2, 147 links, 146 joints
Links:
- removed link GLDistanceSensor1_Link
- removed link GLDistanceSensor2_Link
- removed link GLF1Base_Link
- removed link GLF1DistanceSensorDistal1_Link
- removed link GLF1DistanceSensorDistal2_Link
- removed link GLF1Gear_Link
- removed link GLF1ProximalBar_Link
- removed link GLF1ProximalSegment_Link
- removed link GLF1TopSegment_Link
- removed link GLF1TouchSensorDistal_Link
- removed link GLF1TouchSensorIntermedial_Link
- removed link GLF1TouchSensor_FingerProximal_Link
- removed link GLF2Base_Link
- removed link GLF2DistanceSensorDistal1_Link
- removed link GLF2DistanceSensorDistal2_Link
- removed link GLF2Gear_Link
- removed link GLF2ProximalBar_Link
- removed link GLF2ProximalSegment_Link
- removed link GLF2TopSegment_Link
- removed link GLF2TouchSensorDistal_Link
- removed link GLF2TouchSensorIntermedial_Link
- removed link GLF2TouchSensor_FingerProximal_Link
- removed link GLF3Base_Link
- removed link GLF3DistanceSensorDistal1_Link
- removed link GLF3DistanceSensorDistal2_Link
- removed link GLF3Gear_Link
- removed link GLF3ProximalBar_Link
- removed link GLF3ProximalSegment_Link
- removed link GLF3TopSegment_Link
- removed link GLF3TouchSensorDistal_Link
- removed link GLF3TouchSensorIntermedial_Link
- removed link GLF3TouchSensor_FingerProximal_Link
- removed link GLF4Base_Link
- removed link GLF4DistanceSensorDistal1_Link
- removed link GLF4DistanceSensorDistal2_Link
- removed link GLF4Gear_Link
- removed link GLF4ProximalBar_Link
- removed link GLF4ProximalSegment_Link
- removed link GLF4TopSegment_Link
- removed link GLF4TouchSensorDistal_Link
- removed link GLF4TouchSensorIntermedial_Link
- removed link GLF4TouchSensor_FingerProximal_Link
- removed link GLIMU_Link
- removed link GLThumb_Link
- removed link GRF1Base_Link
- removed link GRF1DistanceSensorDistal1_Link
- removed link GRF1DistanceSensorDistal2_Link
- removed link GRF1Gear_Link
- removed link GRF1ProximalBar_Link
- removed link GRF1ProximalSegment_Link
- removed link GRF1TopSegment_Link
- removed link GRF1TouchSensorDistal_Link
- removed link GRF1TouchSensorIntermedial_Link
- removed link GRF1TouchSensor_FingerProximal_Link
- removed link GRF2Base_Link
- removed link GRF2DistanceSensorDistal1_Link
- removed link GRF2DistanceSensorDistal2_Link
- removed link GRF2Gear_Link
- removed link GRF2ProximalBar_Link
- removed link GRF2ProximalSegment_Link
- removed link GRF2TopSegment_Link
- removed link GRF2TouchSensorDistal_Link
- removed link GRF2TouchSensorIntermedial_Link
- removed link GRF2TouchSensor_FingerProximal_Link
- removed link GRIMU_Link
- added link platform_Link, mass 98.726; collision mesh filename=../meshes/lfs-stl/base_link_convexhull.stl scale=1.0 1.0 1.0; visual mesh filename=../meshes/lfs-stl/base_link.stl
- link ALBase_Link: geometry collision mesh filename=../meshes/lfs-stl/ALBase_Link_convexhull.stl scale=1.0 1.0 1.0; visual mesh filename=../meshes/lfs-stl/ALBase_Link.stl
- link ALElbowAct_Link: geometry collision mesh filename=../meshes/lfs-stl/ALElbow_Act_Link_convexhull.stl scale=1.0 1.0 1.0; visual mesh filename=../meshes/lfs-stl/ALElbow_Act_Link.stl
- link ALElbowB11_Link: geometry collision mesh filename=../meshes/lfs-stl/ALElbow_B11_Link_convexhull.stl scale=1.0 1.0 1.0; visual mesh filename=../meshes/lfs-stl/ALElbow_B11_Link.stl
- link ALElbow_Link: geometry collision mesh filename=../meshes/lfs-stl/ALElbow_Link_convexhull.stl scale=1.0 1.0 1.0; visual mesh filename=../meshes/lfs-stl/ALElbow_Link.stl
- link ALShoulder1_Link: geometry collision mesh filename=../meshes/lfs-stl/ALShoulder1_Link_convexhull.stl scale=1.0 1.0 1.0; visual mesh filename=../meshes/lfs-stl/ALShoulder1_Link.stl
- link ALShoulder2_Link: geometry collision mesh filename=../meshes/lfs-stl/ALShoulder2_Link_convexhull.stl scale=1.0 1.0 1.0; visual mesh filename=../meshes/lfs-stl/ALShoulder2_Link.stl
- link ALShoulder3_Link: geometry collision mesh filename=../meshes/lfs-stl/ALShoulder3_Link_convexhull.stl scale=1.0 1.0 1.0; visual mesh filename=../meshes/lfs-stl/ALShoulder3_Link.stl
- link ALWristAL1_Link: geometry collision mesh filename=../meshes/lfs-stl/ALWrist_AL1_Link_convexhull.stl scale=1.0 1.0 1.0; visual mesh filename=../meshes/lfs-stl/ALWrist_AL1_Link.stl
- link ALWristAR1_Link: geometry collision mesh filename=../meshes/lfs-stl/ALWrist_AR1_Link_convexhull.stl scale=1.0 1.0 1.0; visual mesh filename=../meshes/lfs-stl/ALWrist_AR1_Link.stl
- link ALWristActL_Link: geometry collision mesh filename=../meshes/lfs-stl/ALWrist_ActL_Link_convexhull.stl scale=1.0 1.0 1.0; visual mesh filename=../meshes/lfs-stl/ALWrist_ActL_Link.stl
- link ALWristActR_Link: geometry collision mesh filename=../meshes/lfs-stl/ALWrist_ActR_Link_convexhull.stl scale=1.0 1.0 1.0; visual mesh filename=../meshes/lfs-stl/ALWrist_ActR_Link.stl
- link ALWristBL0_Link: mass 1e-05 -> 0.0
- link ALWristBL1_Link: geometry collision mesh filename=../meshes/lfs-stl/ALWrist_BL1_Link_convexhull.stl scale=1.0 1.0 1.0; visual mesh filename=../meshes/lfs-stl/ALWrist_BL1_Link.stl
- link ALWristBL2_Link: geometry collision mesh filename=../meshes/lfs-stl/ALWrist_BL2_Link_convexhull.stl scale=1.0 1.0 1.0; visual mesh filename=../meshes/lfs-stl/ALWrist_BL2_Link.stl
- link ALWristBL3_Link: geometry collision mesh filename=../meshes/lfs-stl/ALWrist_BL3_Link_convexhull.stl scale=1.0 1.0 1.0; visual mesh filename=../meshes/lfs-stl/ALWrist_BL3_Link.stl
- link ALWristBL4_Link: geometry collision mesh filename=../meshes/lfs-stl/ALWrist_BL4_Link_convexhull.stl scale=1.0 1.0 1.0; visual mesh filename=../meshes/lfs-stl/ALWrist_BL4_Link.stl
- link ALWristBR0_Link: mass 1e-05 -> 0.0
- link ALWristBR1_Link: geometry collision mesh filename=../meshes/lfs-stl/ALWrist_BR1_Link_convexhull.stl scale=1.0 1.0 1.0; visual mesh filename=../meshes/lfs-stl/ALWrist_BR1_Link.stl
- link ALWristBR2_Link: geometry collision mesh filename=../meshes/lfs-stl/ALWrist_BR2_Link_convexhull.stl scale=1.0 1.0 1.0; visual mesh filename=../meshes/lfs-stl/ALWrist_BR2_Link.stl
- link ALWristBR3_Link: geometry collision mesh filename=../meshes/lfs-stl/ALWrist_BR3_Link_convexhull.stl scale=1.0 1.0 1.0; visual mesh filename=../meshes/lfs-stl/ALWrist_BR3_Link.stl
- link ALWristBR4_Link: geometry collision mesh filename=../meshes/lfs-stl/ALWrist_BR4_Link_convexhull.stl scale=1.0 1.0 1.0; visual mesh filename=../meshes/lfs-stl/ALWrist_BR4_Link.stl
- link ALWristBase_Link: geometry collision mesh filename=../meshes/lfs-stl/ALWrist_Base_Link_convexhull.stl scale=1.0 1.0 1.0; visual mesh filename=../meshes/lfs-stl/ALWrist_Base_Link.stl
- link ALWristFT_Link: geometry collision mesh filename=../meshes/lfs-stl/ALWristFT_Link_convexhull.stl scale=1.0 1.0 1.0; visual mesh filename=../meshes/lfs-stl/ALWristFT_Link.stl
- link ALWristPitch_Link: geometry collision mesh filename=../meshes/lfs-stl/ALWristPitch_Link_convexhull.stl scale=1.0 1.0 1.0; visual mesh filename=../meshes/lfs-stl/ALWristPitch_Link.stl
- link ALWristRoll_Link: mass 2e-05 -> 0.0
- link ALWristRoot_Link: geometry collision mesh filename=../meshes/lfs-stl/ALWrist_Root_Link_convexhull.stl scale=1.0 1.0 1.0; visual mesh filename=../meshes/lfs-stl/ALWrist_Root_Link.stl
- link ALWristYaw_Link: geometry collision mesh filename=../meshes/lfs-stl/ALWristYaw_Link_convexhull.stl scale=1.0 1.0 1.0; visual mesh filename=../meshes/lfs-stl/ALWristYaw_Link.stl
- link ARBase_Link: geometry collision mesh filename=../meshes/lfs-stl/ARBase_Link_convexhull.stl scale=1.0 1.0 1.0; visual mesh filename=../meshes/lfs-stl/ARBase_Link.stl scale=1.0 1.0 1.0
- link ARElbowAct_Link: geometry collision mesh filename=../meshes/lfs-stl/ARElbow_Act_Link_convexhull.stl scale=1.0 1.0 1.0; visual mesh filename=../meshes/lfs-stl/ARElbow_Act_Link.stl scale=1.0 1.0 1.0
- link ARElbowB11_Link: geometry collision mesh filename=../meshes/lfs-stl/ARElbow_B11_Link_convexhull.stl scale=1.0 1.0 1.0; visual mesh filename=../meshes/lfs-stl/ARElbow_B11_Link.stl scale=1.0 1.0 1.0
- link ARElbow_Link: geometry collision mesh filename=../meshes/lfs-stl/ARElbow_Link_convexhull.stl scale=1.0 1.0 1.0; visual mesh filename=../meshes/lfs-stl/ARElbow_Link.stl scale=1.0 1.0 1.0
- link ARShoulder1_Link: geometry collision mesh filename=../meshes/lfs-stl/ARShoulder1_Link_convexhull.stl scale=1.0 1.0 1.0; visual mesh filename=../meshes/lfs-stl/ARShoulder1_Link.stl scale=1.0 1.0 1.0
- link ARShoulder2_Link: geometry collision mesh filename=../meshes/lfs-stl/ARShoulder2_Link_convexhull.stl scale=1.0 1.0 1.0; visual mesh filename=../meshes/lfs-stl/ARShoulder2_Link.stl scale=1.0 1.0 1.0
- link ARShoulder3_Link: geometry collision mesh filename=../meshes/lfs-stl/ARShoulder3_Link_convexhull.stl scale=1.0 1.0 1.0; visual mesh filename=../meshes/lfs-stl/ARShoulder3_Link.stl scale=1.0 1.0 1.0
- link ARWristAL1_Link: mass 0.11027956817212799 -> 0.10112999999999997; geometry collision mesh filename=../meshes/lfs-stl/ARWrist_AR1_Link_convexhull.stl scale=1.0 1.0 1.0; visual mesh filename=../meshes/lfs-stl/ARWrist_AR1_Link.stl scale=1.0 1.0 1.0
- link ARWristAR1_Link: mass 0.10112999999999997 -> 0.11027956817212799; geometry collision mesh filename=../meshes/lfs-stl/ARWrist_AL1_Link_convexhull.stl scale=1.0 1.0 1.0; visual mesh filename=../meshes/lfs-stl/ARWrist_AL1_Link.stl scale=1.0 1.0 1.0
- link ARWristActL_Link: mass 0.022414999999999987 -> 0.022415478206029786; geometry collision mesh filename=../meshes/lfs-stl/ARWrist_ActR_Link_convexhull.stl scale=1.0 1.0 1.0; visual mesh filename=../meshes/lfs-stl/ARWrist_ActR_Link.stl scale=1.0 1.0 1.0
- link ARWristActR_Link: mass 0.022415478206029786 -> 0.022414999999999987; geometry collision mesh filename=../meshes/lfs-stl/ARWrist_ActL_Link_convexhull.stl scale=1.0 1.0 1.0; visual mesh filename=../meshes/lfs-stl/ARWrist_ActL_Link.stl scale=1.0 1.0 1.0
- link ARWristBL0_Link: mass 1e-05 -> 0.0
- link ARWristBL1_Link: geometry collision mesh filename=../meshes/lfs-stl/ARWrist_BR1_Link_convexhull.stl scale=1.0 1.0 1.0; visual mesh filename=../meshes/lfs-stl/ARWrist_BR1_Link.stl scale=1.0 1.0 1.0
- link ARWristBL2_Link: mass 0.003730583331722572 -> 0.0037305447563014613; geometry collision mesh filename=../meshes/lfs-stl/ARWrist_BR2_Link_convexhull.stl scale=1.0 1.0 1.0; visual mesh filename=../meshes/lfs-stl/ARWrist_BR2_Link.stl scale=1.0 1.0 1.0
- link ARWristBL3_Link: mass 0.016343668811119795 -> 0.016343666311700304; geometry collision mesh filename=../meshes/lfs-stl/ARWrist_BR3_Link_convexhull.stl scale=1.0 1.0 1.0; visual mesh filename=../meshes/lfs-stl/ARWrist_BR3_Link.stl scale=1.0 1.0 1.0
- link ARWristBL4_Link: mass 0.0116530368127355 -> 0.011653036812768903; geometry collision mesh filename=../meshes/lfs-stl/ARWrist_BR4_Link_convexhull.stl scale=1.0 1.0 1.0; visual mesh filename=../meshes/lfs-stl/ARWrist_BR4_Link.stl scale=1.0 1.0 1.0
- link ARWristBR0_Link: mass 1e-05 -> 0.0
- link ARWristBR1_Link: geometry collision mesh filename=../meshes/lfs-stl/ARWrist_BL1_Link_convexhull.stl scale=1.0 1.0 1.0; visual mesh filename=../meshes/lfs-stl/ARWrist_BL1_Link.stl scale=1.0 1.0 1.0
- link ARWristBR2_Link: mass 0.0037305447563014613 -> 0.003730583331722572; geometry collision mesh filename=../meshes/lfs-stl/ARWrist_BL2_Link_convexhull.stl scale=1.0 1.0 1.0; visual mesh filename=../meshes/lfs-stl/ARWrist_BL2_Link.stl scale=1.0 1.0 1.0
- link ARWristBR3_Link: mass 0.016343666311700304 -> 0.016343668811119795; geometry collision mesh filename=../meshes/lfs-stl/ARWrist_BL3_Link_convexhull.stl scale=1.0 1.0 1.0; visual mesh filename=../meshes/lfs-stl/ARWrist_BL3_Link.stl scale=1.0 1.0 1.0
- link ARWristBR4_Link: mass 0.011653036812768903 -> 0.0116530368127355; geometry collision mesh filename=../meshes/lfs-stl/ARWrist_BL4_Link_convexhull.stl scale=1.0 1.0 1.0; visual mesh filename=../meshes/lfs-stl/ARWrist_BL4_Link.stl scale=1.0 1.0 1.0
- link ARWristBase_Link: geometry collision mesh filename=../meshes/lfs-stl/ARWrist_Base_Link_convexhull.stl scale=1.0 1.0 1.0; visual mesh filename=../meshes/lfs-stl/ARWrist_Base_Link.stl scale=1.0 1.0 1.0
- link ARWristFT_Link: geometry collision mesh filename=../meshes/lfs-stl/ARWristFT_Link_convexhull.stl scale=1.0 1.0 1.0; visual mesh filename=../meshes/lfs-stl/ARWristFT_Link.stl scale=1.0 1.0 1.0
- link ARWristPitch_Link: geometry collision mesh filename=../meshes/lfs-stl/ARWristPitch_Link_convexhull.stl scale=1.0 1.0 1.0; visual mesh filename=../meshes/lfs-stl/ARWristPitch_Link.stl scale=1.0 1.0 1.0
- link ARWristRoll_Link: mass 2e-05 -> 0.0
- link ARWristRoot_Link: geometry collision mesh filename=../meshes/lfs-stl/ARWrist_Root_Link_convexhull.stl scale=1.0 1.0 1.0; visual mesh filename=../meshes/lfs-stl/ARWrist_Root_Link.stl scale=1.0 1.0 1.0
- link ARWristYaw_Link: geometry collision mesh filename=../meshes/lfs-stl/ARWristYaw_Link_convexhull.stl scale=1.0 1.0 1.0; visual mesh filename=../meshes/lfs-stl/ARWristYaw_Link.stl scale=1.0 1.0 1.0
- link BodyActL_Link: geometry collision mesh filename=../meshes/lfs-stl/Body_ActL_convexhull.stl scale=1.0 1.0 1.0; visual mesh filename=../meshes/lfs-stl/Body_ActL.stl
- link BodyActR_Link: geometry collision mesh filename=../meshes/lfs-stl/Body_ActR_convexhull.stl scale=1.0 1.0 1.0; visual mesh filename=../meshes/lfs-stl/Body_ActR.stl
- link BodyBL1_Link: geometry collision mesh filename=../meshes/lfs-stl/Body_BL1_convexhull.stl scale=1.0 1.0 1.0; visual mesh filename=../meshes/lfs-stl/Body_BL1.stl
- link BodyBL2_Link: geometry collision mesh filename=../meshes/lfs-stl/Body_BL2_convexhull.stl scale=1.0 1.0 1.0; visual mesh filename=../meshes/lfs-stl/Body_BL2.stl
- link BodyBR1_Link: geometry collision mesh filename=../meshes/lfs-stl/Body_BR1_convexhull.stl scale=1.0 1.0 1.0; visual mesh filename=../meshes/lfs-stl/Body_BR1.stl
- link BodyBR2_Link: geometry collision mesh filename=../meshes/lfs-stl/Body_BR2_convexhull.stl scale=1.0 1.0 1.0; visual mesh filename=../meshes/lfs-stl/Body_BR2.stl
- link BodyPitch_Link: geometry collision mesh filename=../meshes/lfs-stl/BodyPitch_convexhull.stl scale=1.0 1.0 1.0; visual mesh filename=../meshes/lfs-stl/BodyPitch.stl
- link BodyRoll_Link: geometry collision mesh filename=../meshes/lfs-stl/BodyRoll_convexhull.stl scale=1.0 1.0 1.0; visual mesh filename=../meshes/lfs-stl/BodyRoll.stl
- link BodyRoot_Link: geometry collision mesh filename=../meshes/lfs-stl/Body_Root_Link_convexhull.stl scale=1.0 1.0 1.0; visual mesh filename=../meshes/lfs-stl/Body_Root_Link.stl
- link BodyYaw_Link: geometry collision mesh filename=../meshes/lfs-stl/BodyYaw_convexhull.stl scale=1.0 1.0 1.0; visual mesh filename=../meshes/lfs-stl/BodyYaw.stl
- link Connector_Body/Leg_left_Link: mass 1e-05 -> 0.0
- link Connector_Body/Leg_right_Link: mass 1e-05 -> 0.0
- link Connector_Body/Torso_Link: mass 9.057619513349467 -> 9.057654141048396; geometry collision mesh filename=../meshes/lfs-stl/Connector_BodyTorso_Link_simplified-full-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 scale=1.0 1.0 1.0; visual mesh filename=../meshes/lfs-stl/Connector_Torso_ArmLeft.stl
- link Connector_Torso/Backpack_Link: geometry collision mesh filename=../meshes/lfs-stl/Connector_Torso_Backpack_convexhull.stl scale=1.0 1.0 1.0; visual mesh filename=../meshes/lfs-stl/Connector_Torso_Backpack.stl
- link GLBase_Link: mass 1.6158618735699422 -> 3.1111163372336628; geometry collision mesh filename=../meshes/lfs-stl/GLBase_Link_simplified-full-urdf_joined_c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 scale=1.0 1.0 1.0; visual mesh filename=../meshes/lfs-stl/F_Gear_Frame.stl
- link GRBase_Link: mass 0.16915002046641558 -> 0.8370142201706786; geometry collision mesh filename=../meshes/lfs-stl/GRBase_Link_simplified-full-urdf_joined_c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 scale=1.0 1.0 1.0; visual mesh filename=../meshes/lfs-stl/2FGripper_BaseFrame.stl
- link HeadActC_Link: geometry collision mesh filename=../meshes/lfs-stl/Head_ActC_convexhull.stl scale=1.0 1.0 1.0; visual mesh filename=../meshes/lfs-stl/Head_ActC.stl
- link HeadActL_Link: geometry collision mesh filename=../meshes/lfs-stl/Head_ActL_convexhull.stl scale=1.0 1.0 1.0; visual mesh filename=../meshes/lfs-stl/Head_ActL.stl
- link HeadActR_Link: geometry collision mesh filename=../meshes/lfs-stl/Head_ActR_convexhull.stl scale=1.0 1.0 1.0; visual mesh filename=../meshes/lfs-stl/Head_ActR.stl
- link HeadBase_Link: geometry collision mesh filename=../meshes/lfs-stl/Head_Base_convexhull.stl scale=1.0 1.0 1.0; visual mesh filename=../meshes/lfs-stl/Head_Base.stl
- link HeadPitch_Link: geometry collision mesh filename=../meshes/lfs-stl/HeadPitch_convexhull.stl scale=1.0 1.0 1.0; visual mesh filename=../meshes/lfs-stl/HeadPitch.stl
- link HeadRoll_Link: geometry collision mesh filename=../meshes/lfs-stl/HeadRoll_convexhull.stl scale=1.0 1.0 1.0; visual mesh filename=../meshes/lfs-stl/HeadRoll.stl
- link HeadYaw_Link: geometry collision mesh filename=../meshes/lfs-stl/HeadYaw_convexhull.stl scale=1.0 1.0 1.0; visual mesh filename=../meshes/lfs-stl/HeadYaw.stl
- link IMU_Body_Link: geometry collision mesh filename=../meshes/lfs-stl/IMU_Body_convexhull.stl scale=1.0 1.0 1.0; visual mesh filename=../meshes/lfs-stl/IMU_Body.stl
- link IMU_Torso_Link: geometry collision mesh filename=../meshes/lfs-stl/IMU_Torso_convexhull.stl scale=1.0 1.0 1.0; visual mesh filename=../meshes/lfs-stl/IMU_Torso.stl
- link RH5v2_Root_Link: geometry collision mesh filename=../meshes/lfs-stl/RH5v2_Root_Link_convexhull.stl scale=1.0 1.0 1.0; visual mesh filename=../meshes/lfs-stl/RH5v2_Root_Link.stl
- link Stereo_Camera_Head_Link: mass 0.163942749569653 -> 0.16394274956965307; geometry collision mesh filename=../meshes/lfs-stl/Stereo_Camera_Head_convexhull.stl scale=1.0 1.0 1.0; visual mesh filename=../meshes/lfs-stl/Stereo_Camera_Head.stl
- link Structure_Sensor_Link: mass 0.35771 -> 0.35771000000000003; geometry collision mesh filename=../meshes/lfs-stl/Structure_Sensor_Torso_convexhull.stl scale=1.0 1.0 1.0; visual mesh filename=../meshes/lfs-stl/Structure_Sensor_Torso.stl
Joints:
- removed joint GLDistanceSensor1
- removed joint GLDistanceSensor2
- removed joint GLF1Base
- removed joint GLF1DistanceSensorDistal1
- removed joint GLF1DistanceSensorDistal2
- removed joint GLF1Gear
- removed joint GLF1ProximalBar
- removed joint GLF1ProximalSegment
- removed joint GLF1TopSegment
- removed joint GLF1TouchSensorDistal
- removed joint GLF1TouchSensorIntermedial
- removed joint GLF1TouchSensor_FingerProximal
- removed joint GLF2Base
- removed joint GLF2DistanceSensorDistal1
- removed joint GLF2DistanceSensorDistal2
- removed joint GLF2Gear
- removed joint GLF2ProximalBar
- removed joint GLF2ProximalSegment
- removed joint GLF2TopSegment
- removed joint GLF2TouchSensorDistal
- removed joint GLF2TouchSensorIntermedial
- removed joint GLF2TouchSensor_FingerProximal
- removed joint GLF3Base
- removed joint GLF3DistanceSensorDistal1
- removed joint GLF3DistanceSensorDistal2
- removed joint GLF3Gear
- removed joint GLF3ProximalBar
- removed joint GLF3ProximalSegment
- removed joint GLF3TopSegment
- removed joint GLF3TouchSensorDistal
- removed joint GLF3TouchSensorIntermedial
- removed joint GLF3TouchSensor_FingerProximal
- removed joint GLF4Base
- removed joint GLF4DistanceSensorDistal1
- removed joint GLF4DistanceSensorDistal2
- removed joint GLF4Gear
- removed joint GLF4ProximalBar
- removed joint GLF4ProximalSegment
- removed joint GLF4TopSegment
- removed joint GLF4TouchSensorDistal
- removed joint GLF4TouchSensorIntermedial
- removed joint GLF4TouchSensor_FingerProximal
- removed joint GLIMU
- removed joint GLThumb
- removed joint GRF1Base
- removed joint GRF1DistanceSensorDistal1
- removed joint GRF1DistanceSensorDistal2
- removed joint GRF1Gear
- removed joint GRF1ProximalBar
- removed joint GRF1ProximalSegment
- removed joint GRF1TopSegment
- removed joint GRF1TouchSensorDistal
- removed joint GRF1TouchSensorIntermedial
- removed joint GRF1TouchSensor_FingerProximal
- removed joint GRF2Base
- removed joint GRF2DistanceSensorDistal1
- removed joint GRF2DistanceSensorDistal2
- removed joint GRF2Gear
- removed joint GRF2ProximalBar
- removed joint GRF2ProximalSegment
- removed joint GRF2TopSegment
- removed joint GRF2TouchSensorDistal
- removed joint GRF2TouchSensorIntermedial
- removed joint GRF2TouchSensor_FingerProximal
- removed joint GRIMU
- added joint platform: type fixed, parent Connector_Body/Leg_right_Link, child platform_Link, origin xyz=0.0 0.0 0.0 rpy=0.0 0.0 0.0
- joint ALElbow: limit lower=-1.832 upper=0.0 effort=400.0 velocity=3.1415926 -> lower=-1.78 upper=0.01 effort=110.13 velocity=7.075
- joint ALElbowAct: limit lower=-1.57 upper=1.57 effort=400.0 velocity=3.1415926 -> lower=-0.119 upper=-0.001 effort=2000.0 velocity=0.266
- joint ALShoulder1: limit lower=-3.141 upper=3.141 effort=400.0 velocity=3.1415926 -> lower=-3.0543 upper=3.0543 effort=157.0 velocity=3.6
- joint ALShoulder2: limit lower=-0.253 upper=1.85 effort=400.0 velocity=3.1415926 -> lower=-0.248 upper=1.845 effort=157.0 velocity=3.6
- joint ALShoulder3: limit lower=-3.141 upper=3.141 effort=400.0 velocity=3.1415926 -> lower=-3.0543 upper=3.0543 effort=28.0 velocity=5.7
- joint ALWristActL: limit lower=-1.57 upper=1.57 effort=400.0 velocity=3.1415926 -> lower=-0.018 upper=0.038 effort=1094.0 velocity=0.2
- joint ALWristActR: limit lower=-1.57 upper=1.57 effort=400.0 velocity=3.1415926 -> lower=-0.018 upper=0.038 effort=1094.0 velocity=0.2
- joint ALWristFT: origin xyz=-1.2399e-05 0.0 0.042748 rpy=0.0 0.0 1.5708 -> xyz=0.0 0.0 0.042748 rpy=0.0 0.0 1.5708
- joint ALWristPitch: limit lower=-0.741 upper=1.75 effort=400.0 velocity=3.1415926 -> lower=-0.7 upper=1.57 effort=43.135 velocity=9.255
- joint ALWristRoll: limit lower=-3.141 upper=3.141 effort=400.0 velocity=3.1415926 -> lower=-3.0543 upper=3.0543 effort=28.0 velocity=5.7
- joint ALWristYaw: limit lower=-0.558 upper=0.593 effort=400.0 velocity=3.1415926 -> lower=-0.475 upper=0.585 effort=44.635 velocity=7.725
- joint ARElbow: limit lower=-1.832 upper=0.0 effort=400.0 velocity=3.1415926 -> lower=-1.78 upper=0.01 effort=110.13 velocity=7.075
- joint ARElbowAct: limit lower=-1.57 upper=1.57 effort=400.0 velocity=3.1415926 -> lower=-0.119 upper=0.001 effort=2000.0 velocity=0.266
- joint ARShoulder1: limit lower=-3.141 upper=3.141 effort=400.0 velocity=3.1415926 -> lower=-3.0543 upper=3.0543 effort=157.0 velocity=3.6
- joint ARShoulder2: limit lower=-0.253 upper=1.85 effort=400.0 velocity=3.1415926 -> lower=-0.248 upper=1.845 effort=157.0 velocity=3.6
- joint ARShoulder3: limit lower=-3.141 upper=3.141 effort=400.0 velocity=3.1415926 -> lower=-3.0543 upper=3.0543 effort=28.0 velocity=5.7
- joint ARWristAL1: origin xyz=0.0155 -0.034 0.178 rpy=-1.553093 0.0 3.141592 -> xyz=-0.0155 0.034 -0.178 rpy=1.5885 0.0 -3.141592
- joint ARWristAR1: origin xyz=-0.0155 -0.034 0.178 rpy=-1.553093 0.0 3.141592 -> xyz=0.0155 0.034 -0.178 rpy=1.5885 0.0 -3.141592
- joint ARWristActL: limit lower=-1.57 upper=1.57 effort=400.0 velocity=3.1415926 -> lower=-0.018 upper=0.038 effort=1094.0 velocity=0.2
- joint ARWristActR: limit lower=-1.57 upper=1.57 effort=400.0 velocity=3.1415926 -> lower=-0.018 upper=0.038 effort=1094.0 velocity=0.2
- joint ARWristBL1: origin xyz=0.0155 0.011 0.032 rpy=0.259193 0.0 3.141592 -> xyz=-0.0155 -0.011 -0.032 rpy=-2.8824 0.0 -3.141592
- joint ARWristBL4: origin xyz=0.027 -0.03 0.0 rpy=-0.141793 0.0 3.141592 -> xyz=-0.027 0.03 0.0 rpy=-2.9998 0.0 8e-06
- joint ARWristBR1: origin xyz=-0.0155 0.011 0.032 rpy=0.259193 0.0 3.141592 -> xyz=0.0155 -0.011 -0.032 rpy=-2.8824 0.0 -3.141592
- joint ARWristBR4: origin xyz=-0.027 -0.03 0.0 rpy=0.141793 0.0 -8e-06 -> xyz=0.027 0.03 0.0 rpy=2.9998 0.0 -3.141592
- joint ARWristBase: origin xyz=0.0 0.0 0.168 rpy=-0.016107 1.570793 3.125485 -> xyz=0.0 0.0 -0.168 rpy=-3.141592 -1.570793 -3.141592
- joint ARWristFT: origin xyz=-1.2e-05 0.0 -0.042748 rpy=3.141593 0.0 1.5708 -> xyz=0.0 0.0 0.042748 rpy=0.0 0.0 -1.5708
- joint ARWristPitch: limit lower=-0.741 upper=1.75 effort=400.0 velocity=3.1415926 -> lower=-0.7 upper=1.57 effort=43.135 velocity=9.255; origin xyz=0.0 0.0 0.0 rpy=-0.0 0.0 -1e-06 -> xyz=0.0 0.0 0.0 rpy=0.0 0.0 1e-06
- joint ARWristRoll: limit lower=-3.141 upper=3.141 effort=400.0 velocity=3.1415926 -> lower=-3.0543 upper=3.0543 effort=28.0 velocity=5.7
- joint ARWristRoot: origin xyz=-0.173 0.0 0.0 rpy=-0.010381 -1.5707 -3.131212 -> xyz=-0.173 0.0 0.0 rpy=3.131212 -1.5707 -3.131212
- joint ARWristYaw: limit lower=-0.558 upper=0.593 effort=400.0 velocity=3.1415926 -> lower=-0.475 upper=0.585 effort=44.635 velocity=7.725; origin xyz=0.0 0.0 0.0 rpy=0.0 0.0 1e-06 -> xyz=0.0 0.0 0.0 rpy=0.0 0.0 -1e-06
- joint BodyActL: limit lower=-1.57 upper=1.57 effort=400.0 velocity=3.1415926 -> lower=-0.0345 upper=0.0442 effort=2716.0 velocity=0.291; origin xyz=0.0 0.0 0.23999 rpy=0.0 0.0 -0.0 -> xyz=0.0 0.0 0.23999 rpy=0.0 0.0 0.0
- joint BodyActR: limit lower=-1.57 upper=1.57 effort=400.0 velocity=3.1415926 -> lower=-0.0345 upper=0.0442 effort=2716.0 velocity=0.291; origin xyz=0.0 0.0 0.23999 rpy=0.0 0.0 -0.0 -> xyz=0.0 0.0 0.23999 rpy=0.0 0.0 0.0
- joint BodyBL2: origin xyz=0.0 0.0 0.0 rpy=0.0 -0.010339 -0.0 -> xyz=0.0 0.0 0.0 rpy=0.0 -0.010339 0.0
- joint BodyBR2: origin xyz=0.0 0.0 0.0 rpy=0.0 -0.010339 -0.0 -> xyz=0.0 0.0 0.0 rpy=0.0 -0.010339 0.0
- joint BodyPitch: limit lower=-0.349 upper=0.527 effort=400.0 velocity=3.1415926 -> lower=-0.34 upper=0.52 effort=400.0 velocity=3.1415926
- joint BodyRoll: limit lower=-0.448 upper=0.448 effort=400.0 velocity=3.1415926 -> lower=-0.44 upper=0.44 effort=400.0 velocity=3.1415926; origin xyz=0.0 0.0 0.0 rpy=0.0 0.0 -0.0 -> xyz=0.0 0.0 0.0 rpy=0.0 0.0 0.0
- joint BodyYaw: limit lower=-3.141 upper=3.141 effort=400.0 velocity=3.1415926 -> lower=-3.0543 upper=3.0543 effort=157.0 velocity=3.6; origin xyz=0.0 0.0 0.0 rpy=0.0 0.0 -0.0 -> xyz=0.0 0.0 0.0 rpy=0.0 0.0 0.0
- joint HeadPitch: limit lower=-0.3 upper=0.35 effort=400.0 velocity=3.1415926 -> lower=-0.3 upper=0.35 effort=8.2 velocity=4.8
- joint HeadRoll: limit lower=-0.45 upper=0.007853981633974483 effort=400.0 velocity=3.1415926 -> lower=-0.45 upper=0.45 effort=8.2 velocity=4.8
- joint HeadYaw: limit lower=-2.1 upper=2.1 effort=400.0 velocity=3.1415926 -> lower=-2.1 upper=2.1 effort=4.1 velocity=4.8
- joint Stereo_Camera_Head: origin xyz=0.0689999999999992 -0.103499999999999 -0.0314985000000005 rpy=-1.5707963267949 0.0 -1.5707963267949 -> xyz=0.069 -0.1035 -0.031499 rpy=-3.141496 -1.5707 -1.570796
- joint Structure_Sensor: origin xyz=0.31589 -0.03825 -0.12041 rpy=7e-06 -0.34907 3.141585 -> xyz=0.31589 0.03825 -0.120411 rpy=2.792523 -4e-05 -1.570892
