Commit message: Update test cases and tutorials

File: models/rh5v2/urdf/rh5v2.urdf (robot description, URDF)
Before this commit: robot RH5v2, 53 links, 52 joints
Joints:
- joint GLF1Gear: type revolute -> fixed
- joint GLF1ProximalSegment: type revolute -> fixed
- joint GLF1TopSegment: type revolute -> fixed
- joint GLF2Gear: type revolute -> fixed
- joint GLF2ProximalSegment: type revolute -> fixed
- joint GLF2TopSegment: type revolute -> fixed
- joint GLF3Gear: type revolute -> fixed
- joint GLF3ProximalSegment: type revolute -> fixed
- joint GLF3TopSegment: type revolute -> fixed
- joint GLF4Gear: type revolute -> fixed
- joint GLF4ProximalSegment: type revolute -> fixed
- joint GLF4TopSegment: type revolute -> fixed
- joint GLThumb: type revolute -> fixed
- joint GRF1Gear: type revolute -> fixed
- joint GRF1ProximalSegment: type revolute -> fixed
- joint GRF1TopSegment: type revolute -> fixed
- joint GRF2Gear: type revolute -> fixed
- joint GRF2ProximalSegment: type revolute -> fixed
- joint GRF2TopSegment: type revolute -> fixed
- joint HeadPitch: type revolute -> fixed
- joint HeadRoll: type revolute -> fixed
- joint HeadYaw: type revolute -> fixed
