Commit message: add comparison of different robot models

File: models/kuka/urdf/kuka_iiwa_with_floating_base.urdf (robot description, URDF)
Before this commit: robot kuka_iiwa, 15 links, 14 joints
Links:
- link link_floating_base_rot_x: mass None -> 4
- link link_floating_base_rot_y: mass None -> 4
- link link_floating_base_trans_x: mass None -> 4
- link link_floating_base_trans_y: mass None -> 4
- link link_floating_base_trans_z: mass None -> 4
- link world: mass None -> 4
