Commit message: Update test cases

File: models/kuka/urdf/kuka_iiwa.urdf (robot description, URDF)
Before this commit: robot kuka_iiwa, 9 links, 8 joints
Links:
- link kuka_lbr_l_link_0: geometry collision mesh filename=../meshes/link_0.stl scale=1.0 1.0 1.0; visual mesh filename=../meshes/link_0.stl
- link kuka_lbr_l_link_1: geometry collision mesh filename=../meshes/link_1.stl scale=1.0 1.0 1.0; visual mesh filename=../meshes/link_1.stl
- link kuka_lbr_l_link_2: geometry collision mesh filename=../meshes/link_2.stl scale=1.0 1.0 1.0; visual mesh filename=../meshes/link_2.stl
- link kuka_lbr_l_link_3: geometry collision mesh filename=../meshes/link_3.stl scale=1.0 1.0 1.0; visual mesh filename=../meshes/link_3.stl
- link kuka_lbr_l_link_4: geometry collision mesh filename=../meshes/link_4.stl scale=1.0 1.0 1.0; visual mesh filename=../meshes/link_4.stl
- link kuka_lbr_l_link_5: geometry collision mesh filename=../meshes/link_5.stl scale=1.0 1.0 1.0; visual mesh filename=../meshes/link_5.stl
- link kuka_lbr_l_link_6: geometry collision mesh filename=../meshes/link_6.stl scale=1.0 1.0 1.0; visual mesh filename=../meshes/link_6.stl
- link kuka_lbr_l_link_7: geometry collision mesh filename=../meshes/link_7.stl scale=1.0 1.0 1.0; visual mesh filename=../meshes/link_7.stl

File: models/kuka/urdf/kuka_iiwa_with_floating_base.urdf (robot description, URDF)
Before this commit: robot kuka_iiwa, 15 links, 14 joints
Links:
- link kuka_lbr_l_link_0: geometry collision mesh filename=../meshes/link_0.stl scale=1.0 1.0 1.0; visual mesh filename=../meshes/link_0.stl
- link kuka_lbr_l_link_1: geometry collision mesh filename=../meshes/link_1.stl scale=1.0 1.0 1.0; visual mesh filename=../meshes/link_1.stl
- link kuka_lbr_l_link_2: geometry collision mesh filename=../meshes/link_2.stl scale=1.0 1.0 1.0; visual mesh filename=../meshes/link_2.stl
- link kuka_lbr_l_link_3: geometry collision mesh filename=../meshes/link_3.stl scale=1.0 1.0 1.0; visual mesh filename=../meshes/link_3.stl
- link kuka_lbr_l_link_4: geometry collision mesh filename=../meshes/link_4.stl scale=1.0 1.0 1.0; visual mesh filename=../meshes/link_4.stl
- link kuka_lbr_l_link_5: geometry collision mesh filename=../meshes/link_5.stl scale=1.0 1.0 1.0; visual mesh filename=../meshes/link_5.stl
- link kuka_lbr_l_link_6: geometry collision mesh filename=../meshes/link_6.stl scale=1.0 1.0 1.0; visual mesh filename=../meshes/link_6.stl
- link kuka_lbr_l_link_7: geometry collision mesh filename=../meshes/link_7.stl scale=1.0 1.0 1.0; visual mesh filename=../meshes/link_7.stl

File: models/kuka/urdf/kuka_lbr.urdf (robot description, URDF)
Before this commit: robot kuka_lbr, 59 links, 58 joints
Links:
- link kuka_lbr_l_finger_1_link_0: geometry collision mesh filename=./meshes/collision_finger_1_link_0.stl scale=1.0 1.0 1.0; visual mesh filename=./meshes/visual_finger_1_link_0.stl scale=1.0 1.0 1.0
- link kuka_lbr_l_finger_1_link_1: geometry collision mesh filename=./meshes/collision_finger_1_link_1.stl scale=1.0 1.0 1.0; visual mesh filename=./meshes/visual_finger_1_link_1.stl scale=1.0 1.0 1.0
- link kuka_lbr_l_finger_1_link_2: geometry collision mesh filename=./meshes/collision_finger_1_link_2.stl scale=1.0 1.0 1.0; visual mesh filename=./meshes/visual_finger_1_link_2.stl scale=1.0 1.0 1.0
- link kuka_lbr_l_finger_1_link_3: geometry collision mesh filename=./meshes/collision_finger_1_link_3.stl scale=1.0 1.0 1.0; visual mesh filename=./meshes/visual_finger_1_link_3.stl scale=1.0 1.0 1.0
- link kuka_lbr_l_finger_2_link_0: geometry collision mesh filename=./meshes/collision_finger_2_link_0.stl scale=1.0 1.0 1.0; visual mesh filename=./meshes/visual_finger_2_link_0.stl scale=1.0 1.0 1.0
- link kuka_lbr_l_finger_2_link_1: geometry collision mesh filename=./meshes/collision_finger_2_link_1.stl scale=1.0 1.0 1.0; visual mesh filename=./meshes/visual_finger_2_link_1.stl scale=1.0 1.0 1.0
- link kuka_lbr_l_finger_2_link_2: geometry collision mesh filename=./meshes/collision_finger_2_link_2.stl scale=1.0 1.0 1.0; visual mesh filename=./meshes/visual_finger_2_link_2.stl scale=1.0 1.0 1.0
- link kuka_lbr_l_finger_2_link_3: geometry collision mesh filename=./meshes/collision_finger_2_link_3.stl scale=1.0 1.0 1.0; visual mesh filename=./meshes/visual_finger_2_link_3.stl scale=1.0 1.0 1.0
- link kuka_lbr_l_finger_middle_link_0: geometry collision mesh filename=./meshes/collision_finger_middle_link_0.stl scale=1.0 1.0 1.0; visual mesh filename=./meshes/visual_finger_middle_link_0.stl scale=1.0 1.0 1.0
- link kuka_lbr_l_finger_middle_link_1: geometry collision mesh filename=./meshes/collision_finger_middle_link_1.stl scale=1.0 1.0 1.0; visual mesh filename=./meshes/visual_finger_middle_link_1.stl scale=1.0 1.0 1.0
- link kuka_lbr_l_finger_middle_link_2: geometry collision mesh filename=./meshes/collision_finger_middle_link_2.stl scale=1.0 1.0 1.0; visual mesh filename=./meshes/visual_finger_middle_link_2.stl scale=1.0 1.0 1.0
- link kuka_lbr_l_finger_middle_link_3: geometry collision mesh filename=./meshes/collision_finger_middle_link_3.stl scale=1.0 1.0 1.0; visual mesh filename=./meshes/visual_finger_middle_link_3.stl scale=1.0 1.0 1.0
- link kuka_lbr_l_link_0: geometry collision mesh filename=./meshes/link_0.stl scale=1.0 1.0 1.0; visual mesh filename=./meshes/link_0.stl
- link kuka_lbr_l_link_1: geometry collision mesh filename=./meshes/link_1.stl scale=1.0 1.0 1.0; visual mesh filename=./meshes/link_1.stl
- link kuka_lbr_l_link_2: geometry collision mesh filename=./meshes/link_2.stl scale=1.0 1.0 1.0; visual mesh filename=./meshes/link_2.stl
- link kuka_lbr_l_link_3: geometry collision mesh filename=./meshes/link_3.stl scale=1.0 1.0 1.0; visual mesh filename=./meshes/link_3.stl
- link kuka_lbr_l_link_4: geometry collision mesh filename=./meshes/link_4.stl scale=1.0 1.0 1.0; visual mesh filename=./meshes/link_4.stl
- link kuka_lbr_l_link_5: geometry collision mesh filename=./meshes/link_5.stl scale=1.0 1.0 1.0; visual mesh filename=./meshes/link_5.stl
- link kuka_lbr_l_link_6: geometry collision mesh filename=./meshes/link_6.stl scale=1.0 1.0 1.0; visual mesh filename=./meshes/link_6.stl
- link kuka_lbr_l_link_7: geometry collision mesh filename=./meshes/link_7.stl scale=1.0 1.0 1.0; visual mesh filename=./meshes/link_7.stl
- link kuka_lbr_l_palm_link: geometry collision mesh filename=./meshes/collision_palm.stl scale=1.0 1.0 1.0; visual mesh filename=./meshes/visual_palm.stl scale=1.0 1.0 1.0
- link kuka_lbr_r_finger_1_link_0: geometry collision mesh filename=./meshes/collision_finger_1_link_0.stl scale=1.0 1.0 1.0; visual mesh filename=./meshes/visual_finger_1_link_0.stl scale=1.0 1.0 1.0
- link kuka_lbr_r_finger_1_link_1: geometry collision mesh filename=./meshes/collision_finger_1_link_1.stl scale=1.0 1.0 1.0; visual mesh filename=./meshes/visual_finger_1_link_1.stl scale=1.0 1.0 1.0
- link kuka_lbr_r_finger_1_link_2: geometry collision mesh filename=./meshes/collision_finger_1_link_2.stl scale=1.0 1.0 1.0; visual mesh filename=./meshes/visual_finger_1_link_2.stl scale=1.0 1.0 1.0
- link kuka_lbr_r_finger_1_link_3: geometry collision mesh filename=./meshes/collision_finger_1_link_3.stl scale=1.0 1.0 1.0; visual mesh filename=./meshes/visual_finger_1_link_3.stl scale=1.0 1.0 1.0
- link kuka_lbr_r_finger_2_link_0: geometry collision mesh filename=./meshes/collision_finger_2_link_0.stl scale=1.0 1.0 1.0; visual mesh filename=./meshes/visual_finger_2_link_0.stl scale=1.0 1.0 1.0
- link kuka_lbr_r_finger_2_link_1: geometry collision mesh filename=./meshes/collision_finger_2_link_1.stl scale=1.0 1.0 1.0; visual mesh filename=./meshes/visual_finger_2_link_1.stl scale=1.0 1.0 1.0
- link kuka_lbr_r_finger_2_link_2: geometry collision mesh filename=./meshes/collision_finger_2_link_2.stl scale=1.0 1.0 1.0; visual mesh filename=./meshes/visual_finger_2_link_2.stl scale=1.0 1.0 1.0
- link kuka_lbr_r_finger_2_link_3: geometry collision mesh filename=./meshes/collision_finger_2_link_3.stl scale=1.0 1.0 1.0; visual mesh filename=./meshes/visual_finger_2_link_3.stl scale=1.0 1.0 1.0
- link kuka_lbr_r_finger_middle_link_0: geometry collision mesh filename=./meshes/collision_finger_middle_link_0.stl scale=1.0 1.0 1.0; visual mesh filename=./meshes/visual_finger_middle_link_0.stl scale=1.0 1.0 1.0
- link kuka_lbr_r_finger_middle_link_1: geometry collision mesh filename=./meshes/collision_finger_middle_link_1.stl scale=1.0 1.0 1.0; visual mesh filename=./meshes/visual_finger_middle_link_1.stl scale=1.0 1.0 1.0
- link kuka_lbr_r_finger_middle_link_2: geometry collision mesh filename=./meshes/collision_finger_middle_link_2.stl scale=1.0 1.0 1.0; visual mesh filename=./meshes/visual_finger_middle_link_2.stl scale=1.0 1.0 1.0
- link kuka_lbr_r_finger_middle_link_3: geometry collision mesh filename=./meshes/collision_finger_middle_link_3.stl scale=1.0 1.0 1.0; visual mesh filename=./meshes/visual_finger_middle_link_3.stl scale=1.0 1.0 1.0
- link kuka_lbr_r_link_0: geometry collision mesh filename=./meshes/link_0.stl scale=1.0 1.0 1.0; visual mesh filename=./meshes/link_0.stl
- link kuka_lbr_r_link_1: geometry collision mesh filename=./meshes/link_1.stl scale=1.0 1.0 1.0; visual mesh filename=./meshes/link_1.stl
- link kuka_lbr_r_link_2: geometry collision mesh filename=./meshes/link_2.stl scale=1.0 1.0 1.0; visual mesh filename=./meshes/link_2.stl
- link kuka_lbr_r_link_3: geometry collision mesh filename=./meshes/link_3.stl scale=1.0 1.0 1.0; visual mesh filename=./meshes/link_3.stl
- link kuka_lbr_r_link_4: geometry collision mesh filename=./meshes/link_4.stl scale=1.0 1.0 1.0; visual mesh filename=./meshes/link_4.stl
- link kuka_lbr_r_link_5: geometry collision mesh filename=./meshes/link_5.stl scale=1.0 1.0 1.0; visual mesh filename=./meshes/link_5.stl
- link kuka_lbr_r_link_6: geometry collision mesh filename=./meshes/link_6.stl scale=1.0 1.0 1.0; visual mesh filename=./meshes/link_6.stl
- link kuka_lbr_r_link_7: geometry collision mesh filename=./meshes/link_7.stl scale=1.0 1.0 1.0; visual mesh filename=./meshes/link_7.stl
- link kuka_lbr_r_palm_link: geometry collision mesh filename=./meshes/collision_palm.stl scale=1.0 1.0 1.0; visual mesh filename=./meshes/visual_palm.stl scale=1.0 1.0 1.0

File: models/rh5/urdf/rh5_single_leg.urdf (robot description, URDF)
Before this commit: robot RH5, 13 links, 12 joints
Links:
- link RH5_Root_Link: geometry collision mesh filename=../meshes/RH5_Root_Link.STL scale=1.0 1.0 1.0
