Commit message: Add meshes to models

File: models/rh5/urdf/rh5_floating_base.urdf (robot description, URDF)
Before this commit: robot recupera_exo_and_rh5, 83 links, 82 joints
Links:
- removed link left_exo_elbow
- removed link left_exo_forearm
- removed link left_exo_forearm_ft
- removed link left_exo_hand_ft
- removed link left_exo_handinterface
- removed link left_exo_shoulder_0
- removed link left_exo_shoulder_1_0
- removed link left_exo_upperarm
- removed link left_exo_upperarm_adjustment_contactinterface
- removed link left_exo_upperarm_adjustment_length
- removed link left_exo_upperarm_ft
- removed link object_link
- removed link right_exo_elbow
- removed link right_exo_forearm
- removed link right_exo_forearm_ft
- removed link right_exo_hand_ft
- removed link right_exo_handinterface
- removed link right_exo_shoulder_0
- removed link right_exo_shoulder_1_0
- removed link right_exo_upperarm
- removed link right_exo_upperarm_adjustment_contactinterface
- removed link right_exo_upperarm_adjustment_length
- removed link right_exo_upperarm_ft
- removed link root_link_upper_body_exo
- removed link upperbody_exo_adjustment_1
- removed link upperbody_exo_adjustment_2_left
- removed link upperbody_exo_adjustment_2_right
- removed link upperbody_exo_contact_ft
- added link AL_TCP_Link
- added link Root_Link_rx
- added link Root_Link_ry
- added link Root_Link_x
- added link Root_Link_y
- added link Root_Link_z
- added link world, mass 0.0
- link ALElbow_Link: geometry visual mesh filename=../meshes/ALElbow_Link.STL
- link ALShoulder1_Link: geometry visual mesh filename=../meshes/ALShoulder1_Link.STL
- link ALShoulder2_Link: geometry visual mesh filename=../meshes/ALShoulder2_Link.STL
- link ALShoulder3_Link: geometry collision box size=0.08700039610266685 0.11106326058506966 0.34700000286102295; visual mesh filename=../meshes/ALShoulder3_Link.STL
- link ALWristPitch_Link: geometry visual mesh filename=../meshes/ALWristPitch_Link.STL
- link ALWristRoll_Link: geometry collision box size=0.13932063803076744 0.11817342042922974 0.34249999932944775; visual mesh filename=../meshes/ALWristRoll_Link.STL
- link ALWristYaw_Link: geometry visual mesh filename=../meshes/ALWristYaw_Link.STL
- link ALWrist_FT: geometry collision box size=0.0960712879896164 0.1100204549729824 0.1812121346592903; visual mesh filename=../meshes/ALWrist_FT.STL
- link ARElbow_Link: geometry visual mesh filename=../meshes/ALElbow_Link.STL
- link ARShoulder1_Link: geometry visual mesh filename=../meshes/ARShoulder1_Link.STL
- link ARShoulder2_Link: geometry visual mesh filename=../meshes/ARShoulder2_Link.STL
- link ARShoulder3_Link: geometry collision box size=0.08700039610266685 0.11106326058506966 0.34700000286102295; visual mesh filename=../meshes/ALShoulder3_Link.STL
- link ARWristPitch_Link: geometry visual mesh filename=../meshes/ALWristPitch_Link.STL
- link ARWristRoll_Link: geometry collision box size=0.13932063803076744 0.11817342042922974 0.34249999932944775; visual mesh filename=../meshes/ALWristRoll_Link.STL
- link ARWristYaw_Link: geometry visual mesh filename=../meshes/ALWristYaw_Link.STL
- link ARWrist_FT: geometry collision box size=0.0960712879896164 0.1100204549729824 0.1812121346592903; visual mesh filename=../meshes/ALWrist_FT.STL
- link BodyPitch_Link: geometry visual mesh filename=../meshes/BodyPitch_Link.STL
- link BodyRoll_Link: geometry visual mesh filename=../meshes/BodyRoll_Link.STL
- link BodyYaw_Link: geometry collision box size=0.3599925637245178 0.514311820268631 0.5017095673829317; visual mesh filename=../meshes/BodyYaw_Act1_Link.STL
- link HeadPitch_Link: geometry visual mesh filename=../meshes/HeadPitch_Link.STL
- link HeadRoll_Link: geometry visual mesh filename=../meshes/HeadRoll_Link.STL
- link HeadYaw_Link: geometry collision sphere radius=0.1292259246110916; visual mesh filename=../meshes/HeadYaw_Link.STL
- link LLAnklePitch_Link: geometry visual mesh filename=../meshes/AnklePitch_Link.STL; visual mesh filename=../meshes/Ankle_E11_Link.STL
- link LLAnkleRoll_Link: geometry visual mesh filename=../meshes/AnkleRoll_Link.STL
- link LLAnkle_FT: geometry visual mesh filename=../meshes/FL_FT_Link.STL
- link LLHip1_Link: geometry visual mesh filename=../meshes/LLHip1_Link.STL
- link LLHip2_Link: geometry visual mesh filename=../meshes/Hip3_B11_Link.STL; visual mesh filename=../meshes/LLHip2_Link.STL
- link LLHip3_Link: geometry collision box size=0.12200059773407665 0.15002443346404168 0.474515434996993; visual mesh filename=../meshes/Hip3_Link.STL
- link LLKnee_Link: geometry collision box size=0.5021360367536545 0.12789290770888329 0.11989995092153549; visual mesh filename=../meshes/Ankle_Act1_Link.STL
- link LRAnklePitch_Link: geometry visual mesh filename=../meshes/AnklePitch_Link.STL; visual mesh filename=../meshes/Ankle_E11_Link.STL
- link LRAnkleRoll_Link: geometry visual mesh filename=../meshes/AnkleRoll_Link.STL
- link LRAnkle_FT: geometry visual mesh filename=../meshes/FL_FT_Link.STL
- link LRHip1_Link: geometry visual mesh filename=../meshes/LRHip1_Link.STL
- link LRHip2_Link: geometry visual mesh filename=../meshes/Hip3_B11_Link.STL; visual mesh filename=../meshes/LLHip3_Act1_Link.STL
- link LRHip3_Link: geometry collision box size=0.12200059773407665 0.15002443346404168 0.474515434996993; visual mesh filename=../meshes/Hip3_Link.STL
- link LRKnee_Link: geometry collision box size=0.5021360367536545 0.12789290770888329 0.11989995092153549; visual mesh filename=../meshes/Ankle_Act1_Link.STL
- link RH5_Root_Link: geometry collision box size=0.2746039479970932 0.3261495530605316 0.22715241627884097; visual mesh filename=../meshes/Body_Act1_Link.STL
Joints:
- removed joint left_arm_elbow_joint
- removed joint left_arm_forearm_joint
- removed joint left_arm_shoulder_joint0
- removed joint left_arm_shoulder_joint1
- removed joint left_arm_shoulder_joint2
- removed joint left_exo_handinterface_joint
- removed joint left_exo_upperarm_adjustment_contactinterface_joint
- removed joint left_exo_upperarm_adjustment_length_joint
- removed joint left_forearm_ft
- removed joint left_hand_ft
- removed joint left_upperarm_ft
- removed joint object
- removed joint right_arm_elbow_joint
- removed joint right_arm_forearm_joint
- removed joint right_arm_shoulder_joint0
- removed joint right_arm_shoulder_joint1
- removed joint right_arm_shoulder_joint2
- removed joint right_exo_handinterface_joint
- removed joint right_exo_upperarm_adjustment_contactinterface_joint
- removed joint right_exo_upperarm_adjustment_length_joint
- removed joint right_forearm_ft
- removed joint right_hand_ft
- removed joint right_upperarm_ft
- removed joint root_link_upper_body_exo_to_RH5_Root_Link
- removed joint upperbody_contact_ft
- removed joint upperbody_exo_adjustment_1_joint
- removed joint upperbody_exo_adjustment_2_left_joint
- removed joint upperbody_exo_adjustment_2_right_joint
- added joint AL_TCP: type fixed, parent ALWrist_FT, child AL_TCP_Link, origin xyz=0.01 0.0 0.15 rpy=0 0 0, axis 0.0 0.0 0.0
- added joint floating_base_rot_x: type revolute, parent Root_Link_z, child Root_Link_rx, origin xyz=0 0 0 rpy=0 0 0, axis 1 0 0, limit lower=-1.57 upper=1.57 effort=0 velocity=0
- added joint floating_base_rot_y: type revolute, parent Root_Link_rx, child Root_Link_ry, axis 0 1 0, limit lower=-1.57 upper=1.57 effort=0 velocity=0
- added joint floating_base_rot_z: type revolute, parent Root_Link_ry, child RH5_Root_Link, axis 0 0 1, limit lower=-1.57 upper=1.57 effort=0 velocity=0
- added joint floating_base_trans_x: type prismatic, parent world, child Root_Link_x, origin xyz=0 0 0 rpy=0 0 0, axis 1 0 0, limit lower=-1.57 upper=1.57 effort=0 velocity=0
- added joint floating_base_trans_y: type prismatic, parent Root_Link_x, child Root_Link_y, axis 0 1 0, limit lower=-1.57 upper=1.57 effort=0 velocity=0
- added joint floating_base_trans_z: type prismatic, parent Root_Link_y, child Root_Link_z, axis 0 0 1, limit lower=-1.57 upper=1.57 effort=0 velocity=0
- joint Camera_Left: origin xyz=0.12605 0.0402 0.089608 rpy=0.0 0.0 0.0 -> xyz=0.12605 0.0402 0.089608 rpy=-1.5707999999999998 0 -1.5707999999999998
- joint Camera_Right: origin xyz=0.12605 -0.0402 0.089608 rpy=0.0 0.0 0.0 -> xyz=0.12605 -0.0402 0.089608 rpy=-1.5707999999999998 0 -1.5707999999999998
- joint IMU: origin xyz=0.175 0.0 0.145 rpy=0.0 0 0 -> xyz=0.175 0.0 0.145 rpy=0.0 -1.57079632679 3.14159265359

File: models/rh5/urdf/rh5_legs_floating_base.urdf (robot description, URDF)
Before this commit: robot RH5, 26 links, 25 joints
Links:
- added link Root_Link_rx
- added link Root_Link_ry
- added link Root_Link_x
- added link Root_Link_y
- added link Root_Link_z
- added link world, mass 0.0
Joints:
- added joint floating_base_rot_x: type revolute, parent Root_Link_z, child Root_Link_rx, origin xyz=0 0 0 rpy=0 0 0, axis 1 0 0, limit lower=-1.57 upper=1.57 effort=0 velocity=0
- added joint floating_base_rot_y: type revolute, parent Root_Link_rx, child Root_Link_ry, axis 0 1 0, limit lower=-1.57 upper=1.57 effort=0 velocity=0
- added joint floating_base_rot_z: type revolute, parent Root_Link_ry, child RH5_Root_Link, axis 0 0 1, limit lower=-1.57 upper=1.57 effort=0 velocity=0
- added joint floating_base_trans_x: type prismatic, parent world, child Root_Link_x, origin xyz=0 0 0 rpy=0 0 0, axis 1 0 0, limit lower=-1.57 upper=1.57 effort=0 velocity=0
- added joint floating_base_trans_y: type prismatic, parent Root_Link_x, child Root_Link_y, axis 0 1 0, limit lower=-1.57 upper=1.57 effort=0 velocity=0
- added joint floating_base_trans_z: type prismatic, parent Root_Link_y, child Root_Link_z, axis 0 0 1, limit lower=-1.57 upper=1.57 effort=0 velocity=0
