Commit message: Fix models: Joint names and link names should not be equal

File: models/rh5/urdf/rh5.urdf (robot description, URDF)
Before this commit: robot RH5, 56 links, 55 joints
Joints:
- removed joint FL_SupportCenter
- removed joint FR_SupportCenter
- added joint FL_SupportCenter_joint: type fixed, parent LLAnkle_FT, child FL_SupportCenter, origin xyz=0.03 0.0 0.0444 rpy=3.1416 0.0 0.0, axis 0.0 0.0 0.0
- added joint FR_SupportCenter_joint: type fixed, parent LRAnkle_FT, child FR_SupportCenter, origin xyz=0.03 0.0 0.0444 rpy=3.1416 0.0 0.0, axis 0.0 0.0 0.0

File: models/rh5/urdf/rh5_floating_base.urdf (robot description, URDF)
Before this commit: robot RH5, 62 links, 61 joints
Joints:
- removed joint FL_SupportCenter
- removed joint FR_SupportCenter
- added joint FL_SupportCenter_joint: type fixed, parent LLAnkle_FT, child FL_SupportCenter, origin xyz=0.03 0.0 0.0444 rpy=3.1416 0.0 0.0, axis 0.0 0.0 0.0
- added joint FR_SupportCenter_joint: type fixed, parent LRAnkle_FT, child FR_SupportCenter, origin xyz=0.03 0.0 0.0444 rpy=3.1416 0.0 0.0, axis 0.0 0.0 0.0

File: models/rh5/urdf/rh5_hybrid.urdf (robot description, URDF)
Before this commit: robot RH5, 104 links, 103 joints
Joints:
- removed joint FL_SupportCenter
- removed joint FR_SupportCenter
- added joint FL_SupportCenter_joint: type fixed, parent LLAnkle_FT, child FL_SupportCenter, origin xyz=0.03 0.0 0.0444 rpy=3.1416 0.0 0.0, axis 0.0 0.0 0.0
- added joint FR_SupportCenter_joint: type fixed, parent LRAnkle_FT, child FR_SupportCenter, origin xyz=0.03 0.0 0.0444 rpy=3.1416 0.0 0.0, axis 0.0 0.0 0.0

File: models/rh5/urdf/rh5_legs.urdf (robot description, URDF)
Before this commit: robot RH5, 26 links, 25 joints
Joints:
- removed joint FL_SupportCenter
- removed joint FR_SupportCenter
- added joint FL_SupportCenter_joint: type fixed, parent LLAnkle_FT, child FL_SupportCenter, origin xyz=0.03 0.0 0.0444 rpy=3.1416 0.0 0.0, axis 0.0 0.0 0.0
- added joint FR_SupportCenter_joint: type fixed, parent LRAnkle_FT, child FR_SupportCenter, origin xyz=0.03 0.0 0.0444 rpy=3.1416 0.0 0.0, axis 0.0 0.0 0.0

File: models/rh5/urdf/rh5_legs_floating_base.urdf (robot description, URDF)
Before this commit: robot RH5, 32 links, 31 joints
Joints:
- removed joint FL_SupportCenter
- removed joint FR_SupportCenter
- added joint FL_SupportCenter_joint: type fixed, parent LLAnkle_FT, child FL_SupportCenter, origin xyz=0.03 0.0 0.0444 rpy=3.1416 0.0 0.0, axis 0.0 0.0 0.0
- added joint FR_SupportCenter_joint: type fixed, parent LRAnkle_FT, child FR_SupportCenter, origin xyz=0.03 0.0 0.0444 rpy=3.1416 0.0 0.0, axis 0.0 0.0 0.0

File: models/rh5/urdf/rh5_legs_hybrid.urdf (robot description, URDF)
Before this commit: robot RH5, 51 links, 50 joints
Joints:
- removed joint FL_SupportCenter
- removed joint FR_SupportCenter
- added joint FL_SupportCenter_joint: type fixed, parent LLAnkle_FT, child FL_SupportCenter, origin xyz=0.03 0.0 0.0444 rpy=3.1416 0.0 0.0, axis 0.0 0.0 0.0
- added joint FR_SupportCenter_joint: type fixed, parent LRAnkle_FT, child FR_SupportCenter, origin xyz=0.03 0.0 0.0444 rpy=3.1416 0.0 0.0, axis 0.0 0.0 0.0

File: models/rh5/urdf/rh5_single_leg.urdf (robot description, URDF)
Before this commit: robot RH5, 13 links, 12 joints
Joints:
- removed joint FL_SupportCenter
- added joint FL_SupportCenter_joint: type fixed, parent LLAnkle_FT, child FL_SupportCenter, origin xyz=0.03 0.0 0.0444 rpy=3.1416 0.0 0.0, axis 0.0 0.0 0.0

File: models/rh5/urdf/rh5_single_leg_fixed.urdf (robot description, URDF)
Before this commit: robot RH5, 14 links, 13 joints
Joints:
- removed joint FL_SupportCenter
- added joint FL_SupportCenter_joint: type fixed, parent LLAnkle_FT, child FL_SupportCenter, origin xyz=0.03 0.0 0.0444 rpy=3.1416 0.0 0.0, axis 0.0 0.0 0.0

File: models/rh5/urdf/rh5_single_leg_hybrid.urdf (robot description, URDF)
Before this commit: robot RH5, 26 links, 25 joints
Joints:
- removed joint FL_SupportCenter
- added joint FL_SupportCenter_joint: type fixed, parent LLAnkle_FT, child FL_SupportCenter, origin xyz=0.03 0.0 0.0444 rpy=3.1416 0.0 0.0, axis 0.0 0.0 0.0
