Commit message: Fix python bindings

File: models/rh5/urdf/rh5_single_leg.urdf (robot description, URDF)
Before this commit: robot RH5, 13 links, 12 joints
Joints:
- removed joint LLAnkle_FT
- added joint LLAnkle_FT_joint: type fixed, parent LLAnklePitch_Link, child LLAnkle_FT, origin xyz=0.0 0.0 -0.058972 rpy=-3.1416 0.0 -1.2151e-16, axis 0.0 0.0 0.0
