Commit message: Fix test case: Joint Limits in URDF were invalid

File: models/rh5/urdf/rh5_single_leg_hybrid.urdf (robot description, URDF)
Before this commit: robot RH5, 26 links, 25 joints
Joints:
- joint LLHip3_Act1: limit lower=0 upper=0 effort=0.0 velocity=0.0 -> lower=-0.0255 upper=0.1335 effort=3000.0 velocity=0.175

Commit message: Fix urdf

File: models/rh5/urdf/rh5_single_leg_hybrid.urdf (robot description, URDF)
Before this commit: robot RH5, 26 links, 25 joints
Joints:
- joint LLHip1: origin xyz=0.0735 0.11044 0.014269 rpy=8.0247e-16 0.2618 -1.5708 -> xyz=0 0 0 rpy=8.0247e-16 0.2618 -1.5708

Commit message: Fix path in URDF model

File: models/rh5/urdf/rh5_single_leg_hybrid.urdf (robot description, URDF)
Before this commit: robot RH5, 26 links, 25 joints
Links:
- link RH5_Root_Link: geometry collision mesh filename=../meshes/RH5_Root_Link.STL scale=1.0 1.0 1.0
