Commit message: Pass robot model to tasks for simplicity of use

File: models/rh5/urdf/rh5_legs.urdf (robot description, URDF)
Before this commit: robot RH5, 26 links, 25 joints
Joints:
- removed joint LLAnkle_FT
- removed joint LRAnkle_FT
- added joint LLAnkle_FT_joint: type fixed, parent LLAnklePitch_Link, child LLAnkle_FT, origin xyz=0.0 0.0 -0.058972 rpy=-3.1416 0.0 -1.2151e-16, axis 0.0 0.0 0.0
- added joint LRAnkle_FT_joint: type fixed, parent LRAnklePitch_Link, child LRAnkle_FT, origin xyz=0.0 0.0 -0.058972 rpy=-3.1416 0.0 -1.2151e-16, axis 0.0 0.0 0.0
