Commit message: Add meshes for rh5v2 model

File: models/rh5v2/raisim/rh5v2.urdf (robot description, URDF)
Before this commit: robot RH5v2, 54 links, 53 joints
Links:
- added link world
- link ALShoulder1_Link: geometry collision sphere radius=0.059044141322374344; visual mesh filename=../meshes/ALShoulder1_Link.stl
- link ALShoulder3_Link: geometry collision cylinder length=0.37510071270897083 radius=0.04989704605643945; visual mesh filename=../meshes/ALElbow_Act_Link.stl
- link ALWristRoll_Link: geometry collision cylinder length=0.19892359808020985 radius=0.051451062143852824; visual mesh filename=../meshes/ALWrist_AL1_Link.stl
- link ARShoulder1_Link: geometry collision sphere radius=0.059044145081229044; visual mesh filename=../meshes/ARShoulder1_Link.stl scale=1.0 1.0 1.0
- link ARShoulder3_Link: geometry collision cylinder length=0.37510067633392874 radius=0.04989704634130358; visual mesh filename=../meshes/ARElbow_Act_Link.stl scale=1.0 1.0 1.0
- link ARWristRoll_Link: geometry collision cylinder length=0.19860603208685698 radius=0.05148203817753268; visual mesh filename=../meshes/ARWrist_AL1_Link.stl scale=1.0 1.0 1.0
- link BodyYaw_Link: geometry collision mesh filename=../meshes/BodyYaw_Link_abstract-urdf_joined_convexhull.obj scale=1.0 1.0 1.0; visual mesh filename=../meshes/BodyYaw.stl
- link GLF1ProximalSegment_Link: geometry collision box size=0.030218173173127905 0.034882865322953094 0.0747403673565936; visual mesh filename=../meshes/F_ProximalSegment_Frame.stl
- link GLF1TopSegment_Link: geometry collision box size=0.026310870976772916 0.02858935493300371 0.07745781389552309; visual mesh filename=../meshes/F_TopSegment_Frame.stl
- link GLF2ProximalSegment_Link: geometry collision box size=0.030218173173127905 0.034882865322953094 0.0747403673565936; visual mesh filename=../meshes/F_ProximalSegment_Frame.stl
- link GLF2TopSegment_Link: geometry collision box size=0.026310870976772916 0.02858935493300371 0.07745781389552309; visual mesh filename=../meshes/F_TopSegment_Frame.stl
- link GLF3ProximalSegment_Link: geometry collision box size=0.030218173173127905 0.034882865322953094 0.0747403673565936; visual mesh filename=../meshes/F_ProximalSegment_Frame.stl
- link GLF3TopSegment_Link: geometry collision box size=0.026310870976772916 0.02858935493300371 0.07745781389552309; visual mesh filename=../meshes/F_TopSegment_Frame.stl
- link GLF4ProximalSegment_Link: geometry collision box size=0.030218173173127905 0.034882865322953094 0.0747403673565936; visual mesh filename=../meshes/F_ProximalSegment_Frame.stl
- link GLF4TopSegment_Link: geometry collision box size=0.026310870976772916 0.02858935493300371 0.07745781389552309; visual mesh filename=../meshes/F_TopSegment_Frame.stl
- link GRF1ProximalSegment_Link: geometry collision box size=0.030218173173127905 0.034882865322953094 0.0747403673565936; visual mesh filename=../meshes/F_ProximalSegment_Frame.stl
- link GRF1TopSegment_Link: geometry collision box size=0.026310870976772916 0.02858935493300371 0.07745781389552309; visual mesh filename=../meshes/F_TopSegment_Frame.stl
- link GRF2ProximalSegment_Link: geometry collision box size=0.030218173173127905 0.034882865322953094 0.0747403673565936; visual mesh filename=../meshes/F_ProximalSegment_Frame.stl
- link GRF2TopSegment_Link: geometry collision box size=0.026310870976772916 0.02858935493300371 0.07745781389552309; visual mesh filename=../meshes/F_TopSegment_Frame.stl
- link HeadBase_Link: geometry collision box size=0.15116204744210632 0.15949007075757243 0.18968096600451853; visual mesh filename=../meshes/Head_ActC.stl
- link HeadYaw_Link: geometry collision box size=0.20200141506883382 0.2099636317811051 0.2599446678014104; visual mesh filename=../meshes/HeadYaw.stl
- link RH5v2_Root_Link: geometry collision mesh filename=../meshes/RH5v2_Root_Link_convexhull.obj scale=1.0 1.0 1.0; visual mesh filename=../meshes/Body_ActL.stl
- link Structure_Sensor_Link: geometry collision box size=0.028000000898483875 0.029504660516651193 0.119540258088699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; visual mesh filename=../meshes/Structure_Sensor_Torso.stl
- link platform_Link: geometry collision mesh filename=../meshes/base_link_convexhull.obj scale=1.0 1.0 1.0; visual mesh filename=../meshes/base_link.stl
Joints:
- added joint base_joint: type fixed, parent world, child RH5v2_Root_Link, origin xyz=0 0 0 rpy=0 0 0

File: models/rh5v2/urdf/rh5v2_hybrid.urdf (robot description, URDF)
Before this commit: robot RH5v2, 83 links, 82 joints
Links:
- link ALBase_Link: geometry collision mesh filename=../meshes/ALBase_Link_convexhull.stl scale=1.0 1.0 1.0; visual mesh filename=../meshes/ALBase_Link.stl
- link ALElbowAct_Link: geometry collision mesh filename=../meshes/ALElbow_Act_Link_convexhull.stl scale=1.0 1.0 1.0; visual mesh filename=../meshes/ALElbow_Act_Link.stl
- link ALElbowB11_Link: geometry collision mesh filename=../meshes/ALElbow_B11_Link_convexhull.stl scale=1.0 1.0 1.0; visual mesh filename=../meshes/ALElbow_B11_Link.stl
- link ALElbow_Link: geometry collision mesh filename=../meshes/ALElbow_Link_convexhull.stl scale=1.0 1.0 1.0; visual mesh filename=../meshes/ALElbow_Link.stl
- link ALShoulder1_Link: geometry collision mesh filename=../meshes/ALShoulder1_Link_convexhull.stl scale=1.0 1.0 1.0; visual mesh filename=../meshes/ALShoulder1_Link.stl
- link ALShoulder2_Link: geometry collision mesh filename=../meshes/ALShoulder2_Link_convexhull.stl scale=1.0 1.0 1.0; visual mesh filename=../meshes/ALShoulder2_Link.stl
- link ALShoulder3_Link: geometry collision mesh filename=../meshes/ALShoulder3_Link_convexhull.stl scale=1.0 1.0 1.0; visual mesh filename=../meshes/ALShoulder3_Link.stl
- link ALWristAL1_Link: geometry collision mesh filename=../meshes/ALWrist_AL1_Link_convexhull.stl scale=1.0 1.0 1.0; visual mesh filename=../meshes/ALWrist_AL1_Link.stl
- link ALWristAR1_Link: geometry collision mesh filename=../meshes/ALWrist_AR1_Link_convexhull.stl scale=1.0 1.0 1.0; visual mesh filename=../meshes/ALWrist_AR1_Link.stl
- link ALWristActL_Link: geometry collision mesh filename=../meshes/ALWrist_ActL_Link_convexhull.stl scale=1.0 1.0 1.0; visual mesh filename=../meshes/ALWrist_ActL_Link.stl
- link ALWristActR_Link: geometry collision mesh filename=../meshes/ALWrist_ActR_Link_convexhull.stl scale=1.0 1.0 1.0; visual mesh filename=../meshes/ALWrist_ActR_Link.stl
- link ALWristBL1_Link: geometry collision mesh filename=../meshes/ALWrist_BL1_Link_convexhull.stl scale=1.0 1.0 1.0; visual mesh filename=../meshes/ALWrist_BL1_Link.stl
- link ALWristBL2_Link: geometry collision mesh filename=../meshes/ALWrist_BL2_Link_convexhull.stl scale=1.0 1.0 1.0; visual mesh filename=../meshes/ALWrist_BL2_Link.stl
- link ALWristBL3_Link: geometry collision mesh filename=../meshes/ALWrist_BL3_Link_convexhull.stl scale=1.0 1.0 1.0; visual mesh filename=../meshes/ALWrist_BL3_Link.stl
- link ALWristBL4_Link: geometry collision mesh filename=../meshes/ALWrist_BL4_Link_convexhull.stl scale=1.0 1.0 1.0; visual mesh filename=../meshes/ALWrist_BL4_Link.stl
- link ALWristBR1_Link: geometry collision mesh filename=../meshes/ALWrist_BR1_Link_convexhull.stl scale=1.0 1.0 1.0; visual mesh filename=../meshes/ALWrist_BR1_Link.stl
- link ALWristBR2_Link: geometry collision mesh filename=../meshes/ALWrist_BR2_Link_convexhull.stl scale=1.0 1.0 1.0; visual mesh filename=../meshes/ALWrist_BR2_Link.stl
- link ALWristBR3_Link: geometry collision mesh filename=../meshes/ALWrist_BR3_Link_convexhull.stl scale=1.0 1.0 1.0; visual mesh filename=../meshes/ALWrist_BR3_Link.stl
- link ALWristBR4_Link: geometry collision mesh filename=../meshes/ALWrist_BR4_Link_convexhull.stl scale=1.0 1.0 1.0; visual mesh filename=../meshes/ALWrist_BR4_Link.stl
- link ALWristBase_Link: geometry collision mesh filename=../meshes/ALWrist_Base_Link_convexhull.stl scale=1.0 1.0 1.0; visual mesh filename=../meshes/ALWrist_Base_Link.stl
- link ALWristFT_Link: geometry collision mesh filename=../meshes/ALWristFT_Link_convexhull.stl scale=1.0 1.0 1.0; visual mesh filename=../meshes/ALWristFT_Link.stl
- link ALWristPitch_Link: geometry collision mesh filename=../meshes/ALWristPitch_Link_convexhull.stl scale=1.0 1.0 1.0; visual mesh filename=../meshes/ALWristPitch_Link.stl
- link ALWristRoot_Link: geometry collision mesh filename=../meshes/ALWrist_Root_Link_convexhull.stl scale=1.0 1.0 1.0; visual mesh filename=../meshes/ALWrist_Root_Link.stl
- link ALWristYaw_Link: geometry collision mesh filename=../meshes/ALWristYaw_Link_convexhull.stl scale=1.0 1.0 1.0; visual mesh filename=../meshes/ALWristYaw_Link.stl
- link ARBase_Link: geometry collision mesh filename=../meshes/ARBase_Link_convexhull.stl scale=1.0 1.0 1.0; visual mesh filename=../meshes/ARBase_Link.stl scale=1.0 1.0 1.0
- link ARElbowAct_Link: geometry collision mesh filename=../meshes/ARElbow_Act_Link_convexhull.stl scale=1.0 1.0 1.0; visual mesh filename=../meshes/ARElbow_Act_Link.stl scale=1.0 1.0 1.0
- link ARElbowB11_Link: geometry collision mesh filename=../meshes/ARElbow_B11_Link_convexhull.stl scale=1.0 1.0 1.0; visual mesh filename=../meshes/ARElbow_B11_Link.stl scale=1.0 1.0 1.0
- link ARElbow_Link: geometry collision mesh filename=../meshes/ARElbow_Link_convexhull.stl scale=1.0 1.0 1.0; visual mesh filename=../meshes/ARElbow_Link.stl scale=1.0 1.0 1.0
- link ARShoulder1_Link: geometry collision mesh filename=../meshes/ARShoulder1_Link_convexhull.stl scale=1.0 1.0 1.0; visual mesh filename=../meshes/ARShoulder1_Link.stl scale=1.0 1.0 1.0
- link ARShoulder2_Link: geometry collision mesh filename=../meshes/ARShoulder2_Link_convexhull.stl scale=1.0 1.0 1.0; visual mesh filename=../meshes/ARShoulder2_Link.stl scale=1.0 1.0 1.0
- link ARShoulder3_Link: geometry collision mesh filename=../meshes/ARShoulder3_Link_convexhull.stl scale=1.0 1.0 1.0; visual mesh filename=../meshes/ARShoulder3_Link.stl scale=1.0 1.0 1.0
- link ARWristAL1_Link: geometry collision mesh filename=../meshes/ARWrist_AR1_Link_convexhull.stl scale=1.0 1.0 1.0; visual mesh filename=../meshes/ARWrist_AR1_Link.stl scale=1.0 1.0 1.0
- link ARWristAR1_Link: geometry collision mesh filename=../meshes/ARWrist_AL1_Link_convexhull.stl scale=1.0 1.0 1.0; visual mesh filename=../meshes/ARWrist_AL1_Link.stl scale=1.0 1.0 1.0
- link ARWristActL_Link: geometry collision mesh filename=../meshes/ARWrist_ActR_Link_convexhull.stl scale=1.0 1.0 1.0; visual mesh filename=../meshes/ARWrist_ActR_Link.stl scale=1.0 1.0 1.0
- link ARWristActR_Link: geometry collision mesh filename=../meshes/ARWrist_ActL_Link_convexhull.stl scale=1.0 1.0 1.0; visual mesh filename=../meshes/ARWrist_ActL_Link.stl scale=1.0 1.0 1.0
- link ARWristBL1_Link: geometry collision mesh filename=../meshes/ARWrist_BR1_Link_convexhull.stl scale=1.0 1.0 1.0; visual mesh filename=../meshes/ARWrist_BR1_Link.stl scale=1.0 1.0 1.0
- link ARWristBL2_Link: geometry collision mesh filename=../meshes/ARWrist_BR2_Link_convexhull.stl scale=1.0 1.0 1.0; visual mesh filename=../meshes/ARWrist_BR2_Link.stl scale=1.0 1.0 1.0
- link ARWristBL3_Link: geometry collision mesh filename=../meshes/ARWrist_BR3_Link_convexhull.stl scale=1.0 1.0 1.0; visual mesh filename=../meshes/ARWrist_BR3_Link.stl scale=1.0 1.0 1.0
- link ARWristBL4_Link: geometry collision mesh filename=../meshes/ARWrist_BR4_Link_convexhull.stl scale=1.0 1.0 1.0; visual mesh filename=../meshes/ARWrist_BR4_Link.stl scale=1.0 1.0 1.0
- link ARWristBR1_Link: geometry collision mesh filename=../meshes/ARWrist_BL1_Link_convexhull.stl scale=1.0 1.0 1.0; visual mesh filename=../meshes/ARWrist_BL1_Link.stl scale=1.0 1.0 1.0
- link ARWristBR2_Link: geometry collision mesh filename=../meshes/ARWrist_BL2_Link_convexhull.stl scale=1.0 1.0 1.0; visual mesh filename=../meshes/ARWrist_BL2_Link.stl scale=1.0 1.0 1.0
- link ARWristBR3_Link: geometry collision mesh filename=../meshes/ARWrist_BL3_Link_convexhull.stl scale=1.0 1.0 1.0; visual mesh filename=../meshes/ARWrist_BL3_Link.stl scale=1.0 1.0 1.0
- link ARWristBR4_Link: geometry collision mesh filename=../meshes/ARWrist_BL4_Link_convexhull.stl scale=1.0 1.0 1.0; visual mesh filename=../meshes/ARWrist_BL4_Link.stl scale=1.0 1.0 1.0
- link ARWristBase_Link: geometry collision mesh filename=../meshes/ARWrist_Base_Link_convexhull.stl scale=1.0 1.0 1.0; visual mesh filename=../meshes/ARWrist_Base_Link.stl scale=1.0 1.0 1.0
- link ARWristFT_Link: geometry collision mesh filename=../meshes/ARWristFT_Link_convexhull.stl scale=1.0 1.0 1.0; visual mesh filename=../meshes/ARWristFT_Link.stl scale=1.0 1.0 1.0
- link ARWristPitch_Link: geometry collision mesh filename=../meshes/ARWristPitch_Link_convexhull.stl scale=1.0 1.0 1.0; visual mesh filename=../meshes/ARWristPitch_Link.stl scale=1.0 1.0 1.0
- link ARWristRoot_Link: geometry collision mesh filename=../meshes/ARWrist_Root_Link_convexhull.stl scale=1.0 1.0 1.0; visual mesh filename=../meshes/ARWrist_Root_Link.stl scale=1.0 1.0 1.0
- link ARWristYaw_Link: geometry collision mesh filename=../meshes/ARWristYaw_Link_convexhull.stl scale=1.0 1.0 1.0; visual mesh filename=../meshes/ARWristYaw_Link.stl scale=1.0 1.0 1.0
- link BodyActL_Link: geometry collision mesh filename=../meshes/Body_ActL_convexhull.stl scale=1.0 1.0 1.0; visual mesh filename=../meshes/Body_ActL.stl
- link BodyActR_Link: geometry collision mesh filename=../meshes/Body_ActR_convexhull.stl scale=1.0 1.0 1.0; visual mesh filename=../meshes/Body_ActR.stl
- link BodyBL1_Link: geometry collision mesh filename=../meshes/Body_BL1_convexhull.stl scale=1.0 1.0 1.0; visual mesh filename=../meshes/Body_BL1.stl
- link BodyBL2_Link: geometry collision mesh filename=../meshes/Body_BL2_convexhull.stl scale=1.0 1.0 1.0; visual mesh filename=../meshes/Body_BL2.stl
- link BodyBR1_Link: geometry collision mesh filename=../meshes/Body_BR1_convexhull.stl scale=1.0 1.0 1.0; visual mesh filename=../meshes/Body_BR1.stl
- link BodyBR2_Link: geometry collision mesh filename=../meshes/Body_BR2_convexhull.stl scale=1.0 1.0 1.0; visual mesh filename=../meshes/Body_BR2.stl
- link BodyPitch_Link: geometry collision mesh filename=../meshes/BodyPitch_convexhull.stl scale=1.0 1.0 1.0; visual mesh filename=../meshes/BodyPitch.stl
- link BodyRoll_Link: geometry collision mesh filename=../meshes/BodyRoll_convexhull.stl scale=1.0 1.0 1.0; visual mesh filename=../meshes/BodyRoll.stl
- link BodyRoot_Link: geometry collision mesh filename=../meshes/Body_Root_Link_convexhull.stl scale=1.0 1.0 1.0; visual mesh filename=../meshes/Body_Root_Link.stl
- link BodyYaw_Link: geometry collision mesh filename=../meshes/BodyYaw_convexhull.stl scale=1.0 1.0 1.0; visual mesh filename=../meshes/BodyYaw.stl
- link Connector_Body/Torso_Link: geometry collision mesh filename=../meshes/base_link_torso.stl scale=1.0 1.0 1.0; visual mesh filename=../meshes/Connector_Torso_ArmLeft.stl
- link Connector_Torso/Backpack_Link: geometry collision mesh filename=../meshes/Connector_Torso_Backpack_convexhull.stl scale=1.0 1.0 1.0; visual mesh filename=../meshes/Connector_Torso_Backpack.stl
- link GLBase_Link: geometry visual mesh filename=../meshes/F_Gear_Frame.stl; visual mesh filename=../meshes/F_Gear_Frame.stl
- link GRBase_Link: geometry visual mesh filename=../meshes/2FGripper_BaseFrame.stl; visual mesh filename=../meshes/F_Gear_Frame.stl
- link HeadActC_Link: geometry collision mesh filename=../meshes/Head_ActC_convexhull.stl scale=1.0 1.0 1.0; visual mesh filename=../meshes/Head_ActC.stl
- link HeadActL_Link: geometry collision mesh filename=../meshes/Head_ActL_convexhull.stl scale=1.0 1.0 1.0; visual mesh filename=../meshes/Head_ActL.stl
- link HeadActR_Link: geometry collision mesh filename=../meshes/Head_ActR_convexhull.stl scale=1.0 1.0 1.0; visual mesh filename=../meshes/Head_ActR.stl
- link HeadBase_Link: geometry collision mesh filename=../meshes/Head_Base_convexhull.stl scale=1.0 1.0 1.0; visual mesh filename=../meshes/Head_Base.stl
- link HeadPitch_Link: geometry collision mesh filename=../meshes/HeadPitch_convexhull.stl scale=1.0 1.0 1.0; visual mesh filename=../meshes/HeadPitch.stl
- link HeadRoll_Link: geometry collision mesh filename=../meshes/HeadRoll_convexhull.stl scale=1.0 1.0 1.0; visual mesh filename=../meshes/HeadRoll.stl
- link HeadYaw_Link: geometry collision mesh filename=../meshes/HeadYaw_convexhull.stl scale=1.0 1.0 1.0; visual mesh filename=../meshes/HeadYaw.stl
- link IMU_Body_Link: geometry collision mesh filename=../meshes/IMU_Body_convexhull.stl scale=1.0 1.0 1.0; visual mesh filename=../meshes/IMU_Body.stl
- link IMU_Torso_Link: geometry collision mesh filename=../meshes/IMU_Torso_convexhull.stl scale=1.0 1.0 1.0; visual mesh filename=../meshes/IMU_Torso.stl
- link RH5v2_Root_Link: geometry collision mesh filename=../meshes/RH5v2_Root_Link_convexhull.stl scale=1.0 1.0 1.0; visual mesh filename=../meshes/RH5v2_Root_Link.stl
- link Stereo_Camera_Head_Link: geometry collision mesh filename=../meshes/Stereo_Camera_Head_convexhull.stl scale=1.0 1.0 1.0; visual mesh filename=../meshes/Stereo_Camera_Head.stl
- link Structure_Sensor_Link: geometry collision mesh filename=../meshes/Structure_Sensor_Torso_convexhull.stl scale=1.0 1.0 1.0; visual mesh filename=../meshes/Structure_Sensor_Torso.stl
- link platform_Link: geometry collision mesh filename=../meshes/base_link_convexhull.stl scale=1.0 1.0 1.0; visual mesh filename=../meshes/base_link.stl
